File: SW-SMART-HIGH-LOW.kicad_pcb (KiCad board)
At the start: 2 copper layers, 73 x 69 mm, 21 parts, among them IC1 MCP1416, J1 1 CTL IN, SW1 BTS50010-1TAD, SW2 VNB35N07xx-E

Commit message: fit a lot of stuff onto a small board
Parts:
- added C3V0: 10u, Capacitor_SMD:C_0805_2012Metric_Pad1.18x1.45mm_HandSolder, F.Cu at (133.8, 122.2)
- added C3V1: 100n, Capacitor_SMD:C_0603_1608Metric_Pad1.08x0.95mm_HandSolder, F.Cu at (150.6, 97.3)
- added C5V0: 10u, Capacitor_SMD:C_0805_2012Metric_Pad1.18x1.45mm_HandSolder, F.Cu at (128.5, 122.2)
- added C5V1: 100n, Capacitor_SMD:C_0603_1608Metric_Pad1.08x0.95mm_HandSolder, F.Cu at (146.2, 103.6)
- added CNRST1: 100n, Capacitor_SMD:C_0603_1608Metric_Pad1.08x0.95mm_HandSolder, F.Cu at (134.3, 112.2)
- added CSTM1: 4u7, Capacitor_SMD:C_0805_2012Metric_Pad1.18x1.45mm_HandSolder, F.Cu at (132.5, 108.2)
- added CSTM2: 100n, Capacitor_SMD:C_0603_1608Metric_Pad1.08x0.95mm_HandSolder, F.Cu at (134.3, 108.2)
- added CVIN1: 10u, Capacitor_SMD:C_1206_3216Metric_Pad1.33x1.80mm_HandSolder, F.Cu at (123.2, 122.2)
- added J2: SWLINK, PCM_SparkFun-Connector:1x05_P2.54mm_Locking, F.Cu at (139.8, 121.3)
- added R1: 10K, Resistor_SMD:R_0603_1608Metric_Pad0.98x0.95mm_HandSolder, F.Cu at (142.6, 95.7)
- added U1: STM32G0B1KBTx, Package_QFP:LQFP-32_7x7mm_P0.8mm, F.Cu at (140.8, 110.0)
- added U4: MCP2562-E-SN, Package_SO:SOIC-8_3.9x4.9mm_P1.27mm, F.Cu at (146.2, 98.8)
- added VR3V3: NCV1117ST33, PCM_SparkFun-Semiconductor-Standard:SOT-223-3_TabPin2, F.Cu at (132.2, 128.2)
- added VR5V0: NCV1117ST50, PCM_SparkFun-Semiconductor-Standard:SOT-223-3_TabPin2, F.Cu at (123.5, 128.2)
- J1: value 1 CTL IN -> H GND L; footprint Connector_PinHeader_2.54mm:PinHeader_1x05_P2.54mm_Horizontal -> TerminalBlock_Phoenix:TerminalBlock_Phoenix_MKDS-1,5-3-5.08_1x03_P5.08mm_Horizontal
- moved J1 7.83 mm to (146.9, 90.3), turned to 90 degrees
- moved RIN2 4.43 mm to (139.0, 93.0)
- moved CIN1 2.15 mm to (128.2, 100.1)
- moved RIN1 2.15 mm to (128.2, 98.5)
- moved RIS1 2.15 mm to (128.2, 95.4)
- moved RIS_PROT1 2.15 mm to (128.2, 96.9)
Connections:
- J1 pad 1: /SW1IS -> /CAN_H
- J1 pad 2: /LOW_IN -> GND
- J1 pad 3: unconnected-(J1-Pin_3-Pad3) -> /CAN_L
- RIN1 pad 1: /SW1IN -> unconnected-(RIN1-Pad1)
- RIN2 pad 1: /LOW_IN -> unconnected-(RIN2-Pad1)
- RIS_PROT1 pad 1: /SW1IS -> unconnected-(RIS_PROT1-Pad1)
Routing:
- net GND: track 92.6 -> 145.6 mm, vias 68 -> 79
- net +3.3V: track 0.00 -> 18.3 mm
- net /CAN_L: track 0.00 -> 18.0 mm
- net +5V: track 0.00 -> 17.5 mm
- net /SW1IN: track 14.3 -> 0.00 mm
- net /SW1IS: track 10.4 -> 0.00 mm
- net +12V: track 7.99 -> 17.9 mm
- net /LOW_IN: track 7.00 -> 0.00 mm
- net /CAN_H: track 0.00 -> 6.48 mm
- net Net-(IC1-IN): track 5.73 -> 2.75 mm
- net /SW1IS_PD: track 14.0 -> 11.9 mm
- net Net-(SW1-IN): track 11.7 -> 9.56 mm
- net Net-(U4-STBY): track 0.00 -> 1.88 mm
Other:
- board size 73 x 69 mm -> 72 x 69 mm

Commit message: making progress on the layout
Parts:
- moved CAN1 0.52 mm to (146.4, 90.3)
- renumbered J1 to CAN1, J2 to J1
Routing:
- net GND: track 145.6 -> 145.1 mm
- net /CAN_L: track 18.0 -> 18.5 mm
Other:
- board text added: "1"
Changed lines of the file:
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@@
 	(footprint "TerminalBlock_Phoenix:TerminalBlock_Phoenix_MKDS-1,5-3-5.08_1x03_P5.08mm_Horizontal"
 		(layer "F.Cu")
-		(at 146.9225 90.335 90)
+		(at 146.4 90.335 90)
 		(descr "Terminal Block Phoenix MKDS-1,5-3-5.08, 3 pins, pitch 5.08mm, size 15.2x9.8mm, drill diameter 1.3mm, pad diameter 2.6mm, http://www.farnell.com/datasheets/100425.pdf, script-generated using https://gitlab.com/kicad/libraries/kicad-footprint-generator/-/tree/master/scripts/TerminalBlock_Phoenix")
 		(tags "THT Terminal Block Phoenix MKDS-1,5-3-5.08 pitch 5.08mm size 15.2x9.8mm drill 1.3mm pad 2.6mm")
-		(property "Reference" "J1"
-			(at 5.08 -6.32 90)
+		(property "Reference" "CAN1"
+			(at 14.335 -4.8 180)
 			(layer "F.SilkS")
 			(effects
@@
 		)
 		(property "Value" "H GND L"
-			(at 5.08 5.72 90)
-			(layer "F.Fab")
+			(at 5.08 -6.7 90)
+			(layer "F.SilkS")
 			(effects
 				(font
@@
 		(descr "See our tutorial: https://www.sparkfun.com/tutorials/114")
 		(tags "SparkFun Locking Friction Fit PTH Male headers")
-		(property "Reference" "J2"
+		(property "Reference" "J1"
 			(at 0 -1.5875 0)
-			(layer "F.Fab")
+			(layer "F.SilkS")
+			(hide yes)
 			(effects
 				(font
-					(size 0.5 0.5)
+					(size 0.6 0.6)
 					(thickness 0.1)
 				)
@@
 		)
 		(property "Value" "SWLINK"
-			(at 0 1.905 0)
-			(layer "F.Fab")
+			(at 5.16 -2.027 0)
+			(layer "F.SilkS")
 			(effects
 				(font
-					(size 0.5 0.5)
+					(size 0.6 0.6)
 					(thickness 0.1)
 				)
@@
 		)
 	)
+	(gr_line
+		(start 138.5 122.6)
+		(end 138.5 120)
+		(stroke
+			(width 0.1)
+			(type default)
+		)
+		(layer "F.SilkS")
+	)
+	(gr_line
+		(start 151.3 120.1)
+		(end 151.3 122.6)
+		(stroke
+			(width 0.1)
+			(type default)
+		)
+		(layer "F.SilkS")
+	)
+	(gr_line
+		(start 138.5 120)
+		(end 151.3 120.1)
+		(stroke
+			(width 0.1)
+			(type default)
+		)
+		(layer "F.SilkS")
+	)
+	(gr_line
+		(start 151.3 122.6)
+		(end 138.5 122.6)
+		(stroke
+			(width 0.1)
+			(type default)
+		)
+		(layer "F.SilkS")
+	)
 	(gr_rect
 		(start 81 66)
@@
 		)
 	)
+	(gr_text "1"
+		(at 139.6 119.7 0)
+		(layer "F.SilkS")
+		(effects
+			(font
+				(size 0.6 0.6)
+				(thickness 0.1)
+			)
+			(justify left bottom)
+		)
+	)
 	(segment
 		(start 126.2 106.465)
@@
 	)
 	(segment
-		(start 146.8675 85.2)
-		(end 144.8 85.2)
-		(width 0.406)
-		(layer "B.Cu")
-		(net 1)
-	)
-	(segment
 		(start 129 93.75)
 		(end 129 92.75)
@@
 	)
 	(segment
+		(start 144.8 85.2)
+		(end 140.3 80.7)
+		(width 0.406)
+		(layer "B.Cu")
+		(net 1)
+	)
+	(segment
 		(start 115.2 91.59)
 		(end 124.44 91.59)
@@
 	)
 	(segment
+		(start 146.345 85.2)
+		(end 144.8 85.2)
+		(width 0.406)
+		(layer "B.Cu")
+		(net 1)
+	)
+	(segment
 		(start 129 101.5)
 		(end 129 93.75)
@@
 	)
 	(segment
-		(start 140.3 80.7)
-		(end 137.7 80.7)
+		(start 146.4 85.255)
+		(end 146.345 85.2)
 		(width 0.406)
 		(layer "B.Cu")
@@
 	)
 	(segment
-		(start 146.9225 85.255)
-		(end 146.8675 85.2)
-		(width 0.406)
-		(layer "B.Cu")
-		(net 1)
-	)
-	(segment
-		(start 144.8 85.2)
-		(end 140.3 80.7)
+		(start 140.3 80.7)
+		(end 137.7 80.7)
 		(width 0.406)
 		(layer "B.Cu")
@@
 	)
 	(segment
+		(start 146.6 90.535)
+		(end 146.4 90.335)
+		(width 0.254)
+		(layer "F.Cu")
+		(net 44)
+	)
+	(segment
 		(start 145.615 93.385)
-		(end 146.9225 92.0775)
+		(end 146.6 92.4)
 		(width 0.254)
 		(layer "F.Cu")
@@
 	)
 	(segment
-		(start 146.9225 92.0775)
-		(end 146.9225 90.335)
+		(start 146.6 92.4)
+		(end 146.6 90.535)
 		(width 0.254)
 		(layer "F.Cu")
@@
 	)
 	(segment
-		(start 146.885 94.231966)
-		(end 149.2 91.916966)
+		(start 146.9225 80.175)
+		(end 146.4 80.175)
 		(width 0.254)
 		(layer "F.Cu")
@@
 	)
 	(segment
-		(start 149.2 91.916966)
-		(end 149.2 82.4525)
+		(start 149.2 82.4525)
+		(end 146.9225 80.175)
 		(width 0.254)
 		(layer "F.Cu")
@@
 	)
 	(segment
-		(start 149.2 82.4525)
-		(end 146.9225 80.175)
+		(start 146.885 94.231966)
+		(end 149.2 91.916966)
+		(width 0.254)
+		(layer "F.Cu")
+		(net 45)
+	)
+	(segment
+		(start 149.2 91.916966)
+		(end 149.2 82.4525)
 		(width 0.254)
 		(layer "F.Cu")
@@
 		(min_thickness 0.254)
 		(filled_areas_thickness no)
-		(fill
+		(fill yes
 			(thermal_gap 0.5)
 			(thermal_bridge_width 0.5)
@@
 		(min_thickness 0.254)
 		(filled_areas_thickness no)
-		(fill
+		(fill yes
 			(thermal_gap 0.5)
 			(thermal_bridge_width 0.5)

Commit message: needs a bit more work
Parts:
- added J2: USART1, PCM_SparkFun-Connector:1x04_P2.54mm_Locking, F.Cu at (149.6, 114.3)
Routing:
- net GND: track 145.1 -> 191.9 mm
- net +3.3V: track 18.3 -> 40.9 mm, vias 0 -> 1
- net /SWDIO: track 0.00 -> 16.4 mm
- net /SWCLK: track 0.00 -> 16.3 mm, vias 0 -> 1
- net /NRST: track 0.00 -> 13.5 mm
- net /CAN1_RX: track 0.00 -> 10.0 mm
- net /CAN1_TX: track 0.00 -> 8.70 mm
- net /USART1_TX: track 0.00 -> 5.02 mm
- net /USART1_RX: track 0.00 -> 4.67 mm
- net +5V: track 17.5 -> 21.0 mm, vias 0 -> 1
- net +12V: vias 120 -> 127
